Commit message: Transition to Humble from Foxy

File: description/camera.xacro (robot description, xacro)
@@ -5,5 +5,5 @@
         <child link="camera_link"/>
         <!-- <origin xyz="0.218 0 0.052" rpy="0 ${pi/22} 0"/> -->
-        <origin xyz="0.218 0 0.052" rpy="0 0 0"/>
+        <origin xyz="0.218 0 0.052" rpy="0 0.1 0"/>
     </joint>
     <link name="camera_link">

File: description/lidar.xacro (robot description, xacro)
@@ -26,5 +26,5 @@
         <sensor name="laser" type="ray">
             <pose> 0 0 0 0 0 0 </pose>
-            <visualize>true</visualize>
+            <visualize>false</visualize>
             <update_rate>10</update_rate>
             <ray>
